File: dfm17_tmux/tmux/tmux.kicad_sch (KiCad schematic)
At the start: 21 parts, among them U2 STG719, U3 STG719, U4 STG719, U5 STG719, U6 DG636E, U7 STG719, U8 SN74LV4053A

Commit message: update after ohm out
Parts:
- R?: value 2M -> 332K
- R?: value 20k -> 100
- R?: value 20k -> 1k
Changed lines of the file:
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@@
       (effects (font (size 1.27 1.27)) (justify left) hide)
     )
-    (property "Value" "2M" (id 1) (at 118.11 71.1199 0)
+    (property "Value" "332K" (id 1) (at 118.11 69.8499 0)
       (effects (font (size 1.27 1.27)) (justify left))
     )
@@
       (effects (font (size 1.27 1.27)) (justify left) hide)
     )
-    (property "Value" "20k" (id 1) (at 144.78 34.2899 0)
+    (property "Value" "100" (id 1) (at 144.78 33.0199 0)
       (effects (font (size 1.27 1.27)) (justify left))
     )
@@
       (effects (font (size 1.27 1.27)) (justify left) hide)
     )
-    (property "Value" "20k" (id 1) (at 144.78 25.3999 0)
+    (property "Value" "1k" (id 1) (at 144.78 24.1299 0)
       (effects (font (size 1.27 1.27)) (justify left))
     )
@@
     )
     (path "/80c340c3-0db1-48bf-898a-667b52d5b4ea"
-      (reference "R?") (unit 1) (value "2M") (footprint "")
+      (reference "R?") (unit 1) (value "332K") (footprint "")
     )
     (path "/932ef468-f011-4e64-b968-0590c099e22d"
@@
     )
     (path "/abe8c85a-8e96-44c4-b9f6-0aeb61c14d61"
-      (reference "R?") (unit 1) (value "20k") (footprint "")
+      (reference "R?") (unit 1) (value "100") (footprint "")
     )
     (path "/bb98d0a0-ef65-49dd-ba6a-da766456d1a9"
-      (reference "R?") (unit 1) (value "20k") (footprint "")
+      (reference "R?") (unit 1) (value "1k") (footprint "")
     )
     (path "/f638d45d-8eb8-40d3-9829-4d4198684093"
